Commit message: Update forklift.urdf

File: urdf/forklift.urdf (robot description, URDF)
Before this commit: robot forklift, 16 links, 15 joints
Joints:
- removed joint FLwheel
- removed joint FRwheel
- removed joint RLwheel
- removed joint RRwheel
- added joint FL_joint: type continuous, parent base_link, child FL_wheel, origin xyz=1.32 0.235 0.02, axis 0 1 0, limit lower=-3.14 upper=3.14 effort=1000.0 velocity=0.5
- added joint FR_joint: type continuous, parent base_link, child FR_wheel, origin xyz=1.32 -0.29 0.02, axis 0 1 0, limit lower=-3.14 upper=3.14 effort=1000.0 velocity=0.5
- added joint RL_joint: type continuous, parent base_link, child RL_wheel, origin xyz=1.23 0.235 0.02, axis 0 1 0, limit lower=-3.14 upper=3.14 effort=1000.0 velocity=0.5
- added joint RR_joint: type continuous, parent base_link, child RR_wheel, origin xyz=1.23 -0.29 0.02, axis 0 1 0, limit lower=-3.14 upper=3.14 effort=1000.0 velocity=0.5
